File: rs485-moist-sensor.sch (KiCad schematic (older format))
At the start: 31 parts, among them IC1 ATTINY441-SSU, P1 CONN_02X03, P2 CONN_01X04, Q1 Q_PMOS_GSD, U1 SN65HVD72, U2 MCP1702, X1 16MHz

Commit message: New kicad library order
Parts:
- C1, C2, C3, C4, C5, C6, C7, C8, C9: symbol C -> rs485-moist-sensor-rescue:C-RESCUE-rs485-moist-sensor
- D1, D2: symbol DIODESCH -> rs485-moist-sensor-rescue:DIODESCH-RESCUE-rs485-moist-sensor
- D4: symbol TVS-ARRAY -> rs485-moist-sensor-rescue:TVS-ARRAY-RESCUE-rs485-moist-sensor
- IC1: symbol ATTINY441-SSU -> rs485-moist-sensor-rescue:ATTINY441-SSU-RESCUE-rs485-moist-sensor
- MK1, MK2: symbol Mounting_Hole -> rs485-moist-sensor-rescue:Mounting_Hole-RESCUE-rs485-moist-sensor
- P1: symbol CONN_02X03 -> rs485-moist-sensor-rescue:CONN_02X03-RESCUE-rs485-moist-sensor
- P2: symbol CONN_01X04 -> rs485-moist-sensor-rescue:CONN_01X04-RESCUE-rs485-moist-sensor
- Q1: symbol Q_PMOS_GSD-RESCUE-rs485-moist-sensor -> rs485-moist-sensor-rescue:Q_PMOS_GSD-RESCUE-rs485-moist-sensor
- R1, R2, R3, R4, R5, R6, R7, R8, R9: symbol R -> rs485-moist-sensor-rescue:R-RESCUE-rs485-moist-sensor
- TH1: symbol THERMISTOR -> rs485-moist-sensor-rescue:THERMISTOR-RESCUE-rs485-moist-sensor
- U1: symbol SP3481EN-RESCUE-rs485-moist-sensor -> rs485-moist-sensor-rescue:SP3481EN-RESCUE-rs485-moist-sensor
- U2: symbol MCP1702 -> rs485-moist-sensor-rescue:MCP1702-RESCUE-rs485-moist-sensor
- X1: symbol CRYSTAL -> rs485-moist-sensor-rescue:CRYSTAL-RESCUE-rs485-moist-sensor
Connections:
- wire segments 62 -> 73
