File: interconnect/interconnect.kicad_pcb (KiCad board)
At the start: 2 copper layers, 37.5 x 35.5 mm, 5 parts, among them J1 RJ45, J2 RJ45, J3 RJ45

Commit message: Add step models for rj45 connectors
Other:
- net class Default removed
