File: adapter/adapter.kicad_pcb (KiCad board)
At the start: 2 copper layers, 35.5 x 19.5 mm, 7 parts, among them J1 Conn_01x04_Male, J2 RJ45, J3 Conn_01x02_Male

Commit message: Add some adapter and interconnect pics
Parts:
- moved JP3 8.08 mm to (71.5, 49.5), turned to -90 degrees
Connections:
- net Net-(J1-Pad2) renamed /A
- net Net-(J1-Pad3) renamed /B
- net Net-(J2-Pad7) renamed /A/GND
- net Net-(J2-Pad8) renamed /B/VCC
- J1 pad 1: GND -> Net-(J1-Pad1)
- J1 pad 4: Net-(J1-Pad4) -> GND
- JP3 pad 1: Net-(J1-Pad4) -> Net-(J1-Pad1)
Routing:
- net Net-(J1-Pad1): track 0.00 -> 26.4 mm
- net Net-(J1-Pad4): track 7.44 -> 0.00 mm
- net VCC: track 16.4 -> 14.7 mm
- net Net-(J3-Pad1): track 3.91 -> 2.70 mm
Other:
- board text added: "RS485 adapter v1.1 Albertas Mickenas 2020"
- board text removed: "RS485 adapter v1.0 Albertas Mickenas 2020"
