File: adapter-por/adapter-por.kicad_pcb (KiCad board)
At the start: 2 copper layers, 48.5 x 19.5 mm, 21 parts, among them J1 Conn_01x04_Male, J2 RJ45, J3 Conn_01x02_Male, U1 MCP100, U2 MCP2505, U3 SN74LVC1G3157, U4 SN74LVC1G3157

Commit message: POR adapter fixups
Other:
- board text added: "+"
- board text added: "-"
